Commit message: Simulation ok with gazebo

File: jaguar4x4wheel_description/urdf/jaguar4x4wheel.urdf.xacro (robot description, xacro)
@@ -17,4 +17,7 @@
   <!-- Base footprint is on the ground under the robot -->
   <link name="base_footprint"/>
+  <gazebo reference="base_link">
+    <material>Gazebo/Grey</material>
+  </gazebo>
   <!-- Base link is the center of the robot's bottom plate -->
   <link name="base_link">

File: jaguar4x4wheel_description/urdf/wheel.urdf.xacro (robot description, xacro)
@@ -23,4 +23,7 @@
 <robot xmlns:xacro="http://ros.org/wiki/xacro" name="jaguar_wheel">
 	<xacro:macro name="jaguar_wheel" params="wheel_prefix *joint_pose">
+    <gazebo reference="${wheel_prefix}_wheel_link">
+      <material>Gazebo/Black</material>
+    </gazebo>
 		<link name="${wheel_prefix}_wheel_link">
 			<inertial>

File: jaguar4x4wheel_gazebo/urdf/description.gazebo.xacro (robot description, xacro)
@@ -22,6 +22,7 @@
 -->
 <robot name="jaguar4x4wheel_robot_gazebo" xmlns:xacro="http://ros.org/wiki/xacro">
-  <xacro:arg name="laser_enabled" default="true" />
-  <xacro:include filename="$(find jaguar4x4wheel_description)/urdf/jaguar4x4wheel.urdf" />
+  <xacro:arg name="laser_enabled" default="false" />
+  <xacro:arg name="kinect_enabled" default="false" />
+  <xacro:include filename="$(find jaguar4x4wheel_description)/urdf/jaguar4x4wheel.urdf.xacro" />
   <xacro:include filename="$(find jaguar4x4wheel_gazebo)/urdf/jaguar4x4wheel.gazebo.xacro" />
   <!-- Gazebo plugin for ROS Control -->

Commit message: Add laser to description

File: jaguar4x4wheel_description/urdf/jaguar4x4wheel.urdf.xacro (robot description, xacro)
@@ -54,4 +54,14 @@
     <child link="inertial_link" />
   </joint>
+  <!-- IMU Link is the standard mounting position for the UM6 IMU.-->
+  <!-- Can be modified with environment variables in /etc/ros/setup.bash -->
+  <link name="imu_link"/>
+  <joint name="imu_joint" type="fixed">
+    <origin xyz="0.35 0 0.1" rpy="0 -1.5708 3.1416" />
+    <parent link="base_link" />
+    <child link="imu_link" />
+  </joint>
+  <gazebo reference="imu_link">
+  </gazebo>
   <!-- Wheel macros -->
   <xacro:jaguar_wheel wheel_prefix="front_left">
@@ -67,17 +77,27 @@
     <origin xyz="${-wheelbase/2+wheel_x_offset} ${-track/2} ${wheel_vertical_offset}" rpy="0 0 0" />
   </xacro:jaguar_wheel>
-  <!--link name="front_left_wheel">
-    <visual>
-      <geometry>
-        <cylinder length="0.1" radius="${wheel_radius}"/>
-      </geometry>
-      <origin rpy="1.57075 0 0" xyz="0 0 0"/>
-      <material name="black"/>
-    </visual>
-  </link>
-  <joint name="base_to_fl_wheel" type="fixed">
-    <parent link="base_link"/>
-    <child link="front_left_wheel"/>
-    <origin xyz="${wheelbase/2} -${track/2} ${wheel_vertical_offset}"/>
-  </joint-->
+  <xacro:arg name="laser_enabled" default="false" />
+  <xacro:arg name="kinect_enabled" default="false" />
+  <xacro:if value="$(arg laser_enabled)">
+    <!-- Hokuyo UTM-30LX mounted upside down below the body -->
+    <!--<xacro:include filename="$(find urg_node)/urdf/hokuyo_utm30lx.urdf.xacro" />
+    <xacro:hokuyo_utm30lx name="laser0" parent="base_link" ros_topic="scan" update_rate="40" ray_count="1081" min_angle="-135" max_angle="135">
+      <origin xyz="0.35 0.0 0.0" rpy="${M_PI} 0 0"/>
+    </xacro:hokuyo_utm30lx>-->
+    <xacro:include filename="$(find urg_node)/urdf/hokuyo_urg_04lx_ug01_laser.urdf.xacro" />
+    <xacro:hokuyo_urg_04lx_ug01_laser name="laser0" parent="base_link" ros_topic="scan" update_rate="40" min_angle="-135" max_angle="135">
+      <origin xyz="0.35 0.0 0.0" rpy="${M_PI} 0 0"/>
+    </xacro:hokuyo_urg_04lx_ug01_laser>
+  </xacro:if>
+  <xacro:if value="$(arg kinect_enabled)">
+    <xacro:sensor_arch prefix="" parent="base_link">
+      <origin xyz="-0.35 ${base_y_size/2} 0.51" rpy="0 0 -3.14"/>
+    </xacro:sensor_arch>
+    <joint name="kinect_frame_joint" type="fixed">
+      <origin xyz="0 0 0" rpy="0 0.18 3.14" />
+      <parent link="sensor_arch_mount_link"/>
+      <child link="camera_link"/>
+    </joint>
+    <xacro:kinect_camera prefix="camera"/>
+  </xacro:if>
 </robot>

Commit message: Add bringup launch files

File: jaguar4x4wheel_description/urdf/jaguar4x4wheel.urdf.xacro (robot description, xacro)
@@ -54,14 +54,11 @@
     <child link="inertial_link" />
   </joint>
-  <!-- IMU Link is the standard mounting position for the UM6 IMU.-->
-  <!-- Can be modified with environment variables in /etc/ros/setup.bash -->
+  <!-- IMU Link is the standard mounting position for the IMU.-->
   <link name="imu_link"/>
   <joint name="imu_joint" type="fixed">
-    <origin xyz="0.35 0 0.1" rpy="0 -1.5708 3.1416" />
+    <origin xyz="0.35 0 0.1" rpy="0 -${M_PI}/2 ${M_PI}" />
     <parent link="base_link" />
     <child link="imu_link" />
   </joint>
-  <gazebo reference="imu_link">
-  </gazebo>
   <!-- Wheel macros -->
   <xacro:jaguar_wheel wheel_prefix="front_left">
@@ -77,6 +74,4 @@
     <origin xyz="${-wheelbase/2+wheel_x_offset} ${-track/2} ${wheel_vertical_offset}" rpy="0 0 0" />
   </xacro:jaguar_wheel>
-  <xacro:arg name="laser_enabled" default="false" />
-  <xacro:arg name="kinect_enabled" default="false" />
   <xacro:if value="$(arg laser_enabled)">
     <!-- Hokuyo UTM-30LX mounted upside down below the body -->
@@ -90,14 +85,19 @@
     </xacro:hokuyo_urg_04lx_ug01_laser>-->
   </xacro:if>
-  <xacro:if value="$(arg kinect_enabled)">
-    <xacro:sensor_arch prefix="" parent="base_link">
-      <origin xyz="-0.35 ${base_y_size/2} 0.51" rpy="0 0 -3.14"/>
-    </xacro:sensor_arch>
-    <joint name="kinect_frame_joint" type="fixed">
-      <origin xyz="0 0 0" rpy="0 0.18 3.14" />
-      <parent link="sensor_arch_mount_link"/>
-      <child link="camera_link"/>
+  <xacro:if value="$(arg camera_enabled)">
+    <link name="camera_link"/>
+    <joint name="camera_joint" type="fixed">
+      <origin xyz="0.25 0 0.2" rpy="0 ${M_PI} 0" />
+      <parent link="base_link" />
+      <child link="camera_link" />
     </joint>
-    <xacro:kinect_camera prefix="camera"/>
+  </xacro:if>
+  <xacro:if value="$(arg navsat_enabled)">
+    <link name="navsat_link"/>
+    <joint name="navsat_joint" type="fixed">
+      <origin xyz="0.25 0 0.2" rpy="0 0 0" />
+      <parent link="base_link" />
+      <child link="navsat_link" />
+    </joint>
   </xacro:if>
 </robot>

File: jaguar4x4wheel_gazebo/urdf/description.gazebo.xacro (robot description, xacro)
@@ -23,6 +23,6 @@
 <robot name="jaguar4x4wheel_robot_gazebo" xmlns:xacro="http://ros.org/wiki/xacro">
   <xacro:arg name="laser_enabled" default="false" />
-  <xacro:arg name="kinect_enabled" default="false" />
-  <xacro:include filename="$(find jaguar4x4wheel_description)/urdf/jaguar4x4wheel.urdf.xacro" />
+  <xacro:arg name="camera_enabled" default="false" />
+  <xacro:include filename="$(find jaguar4x4wheel_description)/urdf/description.xacro" />
   <xacro:include filename="$(find jaguar4x4wheel_gazebo)/urdf/jaguar4x4wheel.gazebo.xacro" />
   <!-- Gazebo plugin for ROS Control -->

File: jaguar4x4wheel_gazebo/urdf/jaguar4x4wheel.gazebo.xacro (robot description, xacro)
@@ -55,10 +55,10 @@
     </gazebo>
     <xacro:if value="$(arg laser_enabled)">
-      <gazebo reference="sick_bracket_link">
+      <gazebo reference="laser_bracket_link">
         <material>Gazebo/DarkGrey</material>
       </gazebo>
       <xacro:sick_lms100_gazebo prefix="base"/>
     </xacro:if>
-    <xacro:if value="$(arg kinect_enabled)">
+    <xacro:if value="$(arg camera_enabled)">
       <xacro:kinect_camera_gazebo prefix="camera"/>
     </xacro:if>

Commit message: jaguar4x4wheel_base on real robot
Odom value seems ok, but published odom is wrong

File: jaguar4x4wheel_description/urdf/jaguar4x4wheel.urdf.xacro (robot description, xacro)
@@ -57,5 +57,5 @@
   <link name="imu_link"/>
   <joint name="imu_joint" type="fixed">
-    <origin xyz="0.35 0 0.1" rpy="0 -${M_PI}/2 ${M_PI}" />
+    <origin xyz="0.35 0 0.1" rpy="0 -${M_PI/2} ${M_PI}" />
     <parent link="base_link" />
     <child link="imu_link" />

Commit message: [gazebo] turn camera on
Simulate o3m151 tof camera with octomap

File: jaguar4x4wheel_description/urdf/jaguar4x4wheel.urdf.xacro (robot description, xacro)
@@ -88,5 +88,5 @@
     <link name="camera_link"/>
     <joint name="camera_joint" type="fixed">
-      <origin xyz="0.25 0 0.2" rpy="0 ${M_PI} 0" />
+      <origin xyz="0.25 0 0.2" rpy="0 0 0" />
       <parent link="base_link" />
       <child link="camera_link" />

File: jaguar4x4wheel_gazebo/urdf/accessories/kinect_camera.gazebo.xacro (robot description, xacro)
@@ -16,6 +16,6 @@
         <image>
           <format>R8G8B8</format>
-          <width>640</width>
-          <height>480</height>
+          <width>64</width>
+          <height>16</height>
         </image>
         <clip>
@@ -27,5 +27,5 @@
         <cameraName>${prefix}</cameraName>
         <alwaysOn>true</alwaysOn>
-        <updateRate>10</updateRate>
+        <updateRate>25</updateRate>
         <imageTopicName>rgb/image_raw</imageTopicName>
         <depthImageTopicName>depth/image_raw</depthImageTopicName>

Commit message: Test on robot without gps

File: jaguar4x4wheel_description/urdf/jaguar4x4wheel.urdf.xacro (robot description, xacro)
@@ -57,5 +57,5 @@
   <link name="imu_link"/>
   <joint name="imu_joint" type="fixed">
-    <origin xyz="0.35 0 0.1" rpy="0 -${M_PI/2} ${M_PI}" />
+    <origin xyz="0.35 0 0.1" rpy="0 0 0" />
     <parent link="base_link" />
     <child link="imu_link" />
@@ -88,5 +88,5 @@
     <link name="camera_link"/>
     <joint name="camera_joint" type="fixed">
-      <origin xyz="0.25 0 0.2" rpy="0 0 0" />
+      <origin xyz="0.35 0 0.41" rpy="0 0 0" />
       <parent link="base_link" />
       <child link="camera_link" />
@@ -96,5 +96,5 @@
     <link name="navsat_link"/>
     <joint name="navsat_joint" type="fixed">
-      <origin xyz="0.25 0 0.2" rpy="0 0 0" />
+      <origin xyz="0.3 0 0.3" rpy="0 0 0" />
       <parent link="base_link" />
       <child link="navsat_link" />

File: jaguar4x4wheel_gazebo/urdf/accessories/kinect_camera.gazebo.xacro (robot description, xacro)
@@ -30,5 +30,5 @@
         <imageTopicName>rgb/image_raw</imageTopicName>
         <depthImageTopicName>depth/image_raw</depthImageTopicName>
-        <pointCloudTopicName>depth/points</pointCloudTopicName>
+        <pointCloudTopicName>filtered_points</pointCloudTopicName>
         <cameraInfoTopicName>rgb/camera_info</cameraInfoTopicName>
         <depthImageCameraInfoTopicName>depth/camera_info</depthImageCameraInfoTopicName>

Commit message: Made base_footprint parent of base_link frame

File: jaguar4x4wheel_description/urdf/jaguar4x4wheel.urdf.xacro (robot description, xacro)
@@ -37,7 +37,7 @@
   </link>
   <joint name="base_footprint_joint" type="fixed">
-    <origin xyz="0 0 ${wheel_vertical_offset - wheel_radius}" rpy="0 0 0" />
-    <parent link="base_link" />
-    <child link="base_footprint" />
+    <origin xyz="0 0 ${-wheel_vertical_offset + wheel_radius}" rpy="0 0 0" />
+    <child link="base_link" />
+    <parent link="base_footprint" />
   </joint>
   <!-- Interial link stores the robot's inertial information -->

Commit message: jaguar description measures updated

File: jaguar4x4wheel_description/urdf/jaguar4x4wheel.urdf.xacro (robot description, xacro)
@@ -4,15 +4,19 @@
   <property name="M_PI" value="3.14159"/>
   <!-- Base Size -->
-  <property name="base_x_size" value="0.50000" />
+  <property name="base_x_size" value="0.49500" />
   <property name="base_y_size" value="0.37000" />
-  <property name="base_z_size" value="0.17000" />
+  <property name="base_z_size" value="0.16000" />
   <!-- Wheel Mounting Positions -->
   <property name="wheelbase" value="0.35" />
-  <property name="track" value="0.48" />
-  <property name="wheel_vertical_offset" value="-0.06" />
+  <property name="track" value="0.475" />
+  <property name="ground_clearance" value="0.09" />
   <property name="wheel_x_offset" value="-0.02" />
   <!-- Wheel Properties -->
   <property name="wheel_length" value="0.09" />
-  <property name="wheel_radius" value="0.13" />
+  <property name="wheel_radius" value="0.1275" />
+  <!-- LIDAR Properties -->
+  <property name="lidar_ground_clearance" value="0.38" />
+<!--   <property name="lidar_ground_clearance" value="0.33" /> -->
+  <property name="lidar_x_offset" value="0.16" />
   <!-- Base footprint is on the ground under the robot -->
   <link name="base_footprint"/>
@@ -37,5 +41,5 @@
   </link>
   <joint name="base_footprint_joint" type="fixed">
-    <origin xyz="0 0 ${-wheel_vertical_offset + wheel_radius}" rpy="0 0 0" />
+    <origin xyz="0 0 ${ground_clearance + base_z_size/2}" rpy="0 0 0" />
     <child link="base_link" />
     <parent link="base_footprint" />
@@ -63,14 +67,14 @@
   <!-- Wheel macros -->
   <xacro:jaguar_wheel wheel_prefix="front_left">
-    <origin xyz="${wheelbase/2+wheel_x_offset} ${track/2} ${wheel_vertical_offset}" rpy="0 0 0" />
+    <origin xyz="${wheelbase/2+wheel_x_offset} ${track/2} -${base_z_size/2 - wheel_radius + ground_clearance}" rpy="0 0 0" />
   </xacro:jaguar_wheel>
   <xacro:jaguar_wheel wheel_prefix="front_right">
-    <origin xyz="${wheelbase/2+wheel_x_offset} ${-track/2} ${wheel_vertical_offset}" rpy="0 0 0" />
+    <origin xyz="${wheelbase/2+wheel_x_offset} ${-track/2} -${base_z_size/2 - wheel_radius + ground_clearance}" rpy="0 0 0" />
   </xacro:jaguar_wheel>
   <xacro:jaguar_wheel wheel_prefix="rear_left">
-    <origin xyz="${-wheelbase/2+wheel_x_offset} ${track/2} ${wheel_vertical_offset}" rpy="0 0 0" />
+    <origin xyz="${-wheelbase/2+wheel_x_offset} ${track/2} -${base_z_size/2 - wheel_radius + ground_clearance}" rpy="0 0 0" />
   </xacro:jaguar_wheel>
   <xacro:jaguar_wheel wheel_prefix="rear_right">
-    <origin xyz="${-wheelbase/2+wheel_x_offset} ${-track/2} ${wheel_vertical_offset}" rpy="0 0 0" />
+    <origin xyz="${-wheelbase/2+wheel_x_offset} ${-track/2} -${base_z_size/2 - wheel_radius + ground_clearance}" rpy="0 0 0" />
   </xacro:jaguar_wheel>
   <xacro:if value="$(arg laser_enabled)">
@@ -78,10 +82,17 @@
     <xacro:include filename="$(find urg_description)/urdf/hokuyo_utm30lx.urdf.xacro" />
     <xacro:hokuyo_utm30lx name="laser0" parent="base_link" ros_topic="scan" update_rate="40" ray_count="1081" min_angle="-135" max_angle="135">
-      <origin xyz="0.35 0.0 0.0" rpy="${M_PI} 0 0"/>
+      <origin xyz="${lidar_x_offset} 0.0 ${lidar_ground_clearance - base_z_size/2 - wheel_radius}" rpy="${M_PI} 0 0"/>
     </xacro:hokuyo_utm30lx>
-    <!--<xacro:include filename="$(find urg_description)/urdf/hokuyo_urg_04lx_ug01_laser.urdf.xacro" />
+<!--    <xacro:include filename="$(find urg_description)/urdf/hokuyo_urg_04lx_ug01_laser.urdf.xacro" />
     <xacro:hokuyo_urg_04lx_ug01_laser name="laser0" parent="base_link" ros_topic="scan" update_rate="40" min_angle="-135" max_angle="135">
       <origin xyz="0.35 0.0 0.0" rpy="${M_PI} 0 0"/>
     </xacro:hokuyo_urg_04lx_ug01_laser>-->
+<!--       <xacro:include filename="$(find sick_tim)/urdf/sick_tim.urdf.xacro" />
+       <xacro:sick_tim551 name="laser0" ros_topic="scan" />
+        <joint name="laser0_mount_joint" type="fixed">
+            <origin xyz="${lidar_x_offset} 0.0 ${lidar_ground_clearance - base_z_size/2 - wheel_radius}" rpy="${M_PI} 0 0" />
+            <parent link="base_link" />
+            <child link="laser0_mount_link" />
+        </joint>-->
   </xacro:if>
   <xacro:if value="$(arg camera_enabled)">

Commit message: Update jaguar description with sick tim

File: jaguar4x4wheel_description/urdf/jaguar4x4wheel.urdf.xacro (robot description, xacro)
@@ -67,32 +67,32 @@
   <!-- Wheel macros -->
   <xacro:jaguar_wheel wheel_prefix="front_left">
-    <origin xyz="${wheelbase/2+wheel_x_offset} ${track/2} -${base_z_size/2 - wheel_radius + ground_clearance}" rpy="0 0 0" />
+    <origin xyz="${wheelbase/2+wheel_x_offset} ${track/2} ${-base_z_size/2 + wheel_radius - ground_clearance}" rpy="0 0 0" />
   </xacro:jaguar_wheel>
   <xacro:jaguar_wheel wheel_prefix="front_right">
-    <origin xyz="${wheelbase/2+wheel_x_offset} ${-track/2} -${base_z_size/2 - wheel_radius + ground_clearance}" rpy="0 0 0" />
+    <origin xyz="${wheelbase/2+wheel_x_offset} ${-track/2} ${-base_z_size/2 + wheel_radius - ground_clearance}" rpy="0 0 0" />
   </xacro:jaguar_wheel>
   <xacro:jaguar_wheel wheel_prefix="rear_left">
-    <origin xyz="${-wheelbase/2+wheel_x_offset} ${track/2} -${base_z_size/2 - wheel_radius + ground_clearance}" rpy="0 0 0" />
+    <origin xyz="${-wheelbase/2+wheel_x_offset} ${track/2} ${-base_z_size/2 + wheel_radius - ground_clearance}" rpy="0 0 0" />
   </xacro:jaguar_wheel>
   <xacro:jaguar_wheel wheel_prefix="rear_right">
-    <origin xyz="${-wheelbase/2+wheel_x_offset} ${-track/2} -${base_z_size/2 - wheel_radius + ground_clearance}" rpy="0 0 0" />
+    <origin xyz="${-wheelbase/2+wheel_x_offset} ${-track/2} ${-base_z_size/2 + wheel_radius - ground_clearance}" rpy="0 0 0" />
   </xacro:jaguar_wheel>
   <xacro:if value="$(arg laser_enabled)">
     <!-- Hokuyo UTM-30LX mounted upside down below the body -->
-    <xacro:include filename="$(find urg_description)/urdf/hokuyo_utm30lx.urdf.xacro" />
+    <!--<xacro:include filename="$(find urg_description)/urdf/hokuyo_utm30lx.urdf.xacro" />
     <xacro:hokuyo_utm30lx name="laser0" parent="base_link" ros_topic="scan" update_rate="40" ray_count="1081" min_angle="-135" max_angle="135">
       <origin xyz="${lidar_x_offset} 0.0 ${lidar_ground_clearance - base_z_size/2 - wheel_radius}" rpy="${M_PI} 0 0"/>
-    </xacro:hokuyo_utm30lx>
+    </xacro:hokuyo_utm30lx>-->
 <!--    <xacro:include filename="$(find urg_description)/urdf/hokuyo_urg_04lx_ug01_laser.urdf.xacro" />
     <xacro:hokuyo_urg_04lx_ug01_laser name="laser0" parent="base_link" ros_topic="scan" update_rate="40" min_angle="-135" max_angle="135">
       <origin xyz="0.35 0.0 0.0" rpy="${M_PI} 0 0"/>
     </xacro:hokuyo_urg_04lx_ug01_laser>-->
-<!--       <xacro:include filename="$(find sick_tim)/urdf/sick_tim.urdf.xacro" />
-       <xacro:sick_tim551 name="laser0" ros_topic="scan" />
-        <joint name="laser0_mount_joint" type="fixed">
-            <origin xyz="${lidar_x_offset} 0.0 ${lidar_ground_clearance - base_z_size/2 - wheel_radius}" rpy="${M_PI} 0 0" />
-            <parent link="base_link" />
-            <child link="laser0_mount_link" />
-        </joint>-->
+    <xacro:include filename="$(find sick_tim)/urdf/sick_tim.urdf.xacro" />
+    <xacro:sick_tim551 name="laser0" ros_topic="scan" />
+    <joint name="laser0_mount_joint" type="fixed">
+      <origin xyz="${lidar_x_offset} 0.0 ${lidar_ground_clearance - base_z_size/2 - wheel_radius}" rpy="${M_PI} 0 0" />
+      <parent link="base_link" />
+      <child link="laser0_mount_link" />
+    </joint>
   </xacro:if>
   <xacro:if value="$(arg camera_enabled)">
